Commit message: ulol

File: assembly_robot_control/ulol_tf/object_description/chair_urdf_for_real/101350.SLDPRT.urdf (robot description, URDF)
Before this commit: robot chair part4.SLDPRT, 1 links, 0 joints
Links:
- removed link chair part4.SLDPRT
- added link 101350.SLDPRT, mass 0.0014585; collision mesh filename=package://object_description/chair_meshes/101350.SLDPRT.STL; visual mesh filename=package://object_description/chair_meshes/101350.SLDPRT.STL

File: assembly_robot_control/ulol_tf/object_description/chair_urdf_for_real/104322.SLDPRT.urdf (robot description, URDF)
Before this commit: robot chair part4.SLDPRT, 1 links, 0 joints
Links:
- removed link chair part4.SLDPRT
- added link 104322.SLDPRT, mass 0.0017863; collision mesh filename=package://object_description/chair_meshes/104322.SLDPRT.STL; visual mesh filename=package://object_description/chair_meshes/104322.SLDPRT.STL

File: assembly_robot_control/ulol_tf/object_description/chair_urdf_for_real/122620.SLDPRT.urdf (robot description, URDF)
Before this commit: robot chair part4.SLDPRT, 1 links, 0 joints
Links:
- removed link chair part4.SLDPRT
- added link 122620.SLDPRT, mass 0.001497; collision mesh filename=package://object_description/chair_meshes/122620.SLDPRT.STL; visual mesh filename=package://object_description/chair_meshes/122620.SLDPRT.STL

File: assembly_robot_control/ulol_tf/object_description/chair_urdf_for_real/122925.SLDPRT.urdf (robot description, URDF)
Before this commit: robot chair part4.SLDPRT, 1 links, 0 joints
Links:
- removed link chair part4.SLDPRT
- added link 122925.SLDPRT, mass 0.00065266; collision mesh filename=package://object_description/chair_meshes/122925.SLDPRT.STL; visual mesh filename=package://object_description/chair_meshes/122925.SLDPRT.STL

File: assembly_robot_control/ulol_tf/object_description/chair_urdf_for_real/chair_part1.SLDPRT.urdf (robot description, URDF)
Before this commit: robot chair part4.SLDPRT, 1 links, 0 joints
Links:
- removed link chair part4.SLDPRT
- added link chair part1.SLDPRT, mass 1.556; collision mesh filename=package://object_description/chair_meshes/chair part1.SLDPR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; visual mesh filename=package://object_description/chair_meshes/chair part1.SLDPR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

File: assembly_robot_control/ulol_tf/object_description/chair_urdf_for_real/chair_part2.SLDPRT.urdf (robot description, URDF)
Before this commit: robot chair part4.SLDPRT, 1 links, 0 joints
Links:
- removed link chair part4.SLDPRT
- added link chair part2.SLDPRT, mass 0.33374; collision mesh filename=package://object_description/chair_meshes/chair part2.SLDPR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; visual mesh filename=package://object_description/chair_meshes/chair part2.SLDPR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

File: assembly_robot_control/ulol_tf/object_description/chair_urdf_for_real/chair_part3.SLDPRT.urdf (robot description, URDF)
Before this commit: robot chair part4.SLDPRT, 1 links, 0 joints
Links:
- removed link chair part4.SLDPRT
- added link chair part3.SLDPRT, mass 0.26482; collision mesh filename=package://object_description/chair_meshes/chair part3.SLDPR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; visual mesh filename=package://object_description/chair_meshes/chair part3.SLDPR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

File: assembly_robot_control/ulol_tf/object_description/chair_urdf_for_real/chair_part5.SLDPRT.urdf (robot description, URDF)
Before this commit: robot chair part4.SLDPRT, 1 links, 0 joints
Links:
- removed link chair part4.SLDPRT
- added link chair part5.SLDPRT, mass 1.8822; collision mesh filename=package://object_description/chair_meshes/chair part5.SLDPR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; visual mesh filename=package://object_description/chair_meshes/chair part5.SLDPR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

File: assembly_robot_control/ulol_tf/object_description/chair_urdf_for_real/chair_part6.SLDPRT.urdf (robot description, URDF)
Before this commit: robot chair part4.SLDPRT, 1 links, 0 joints
Links:
- removed link chair part4.SLDPRT
- added link chair part6.SLDPRT, mass 1.8822; collision mesh filename=package://object_description/chair_meshes/chair part6.SLDPR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; visual mesh filename=package://object_description/chair_meshes/chair part6.SLDPR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
