Commit message: realsense model update

File: assembly_robot_description/urdf/rob1_gripper.urdf.xacro (robot description, xacro)
@@ -4,4 +4,5 @@
   <xacro:arg name="ur_enabled" default="true"/>
   <xacro:arg name="gripper_enabled" default="true"/>
+  <xacro:arg name="realsense_enabled" default="true"/>
   <xacro:property name="M_PI" value="3.14159"/>
   <!--components-->
@@ -9,4 +10,5 @@
 <!--   <xacro:include filename="$(find ur_description)/urdf/ur5.urdf.xacro" /> -->
   <xacro:include filename="$(find robotiq_2f_85_gripper_visualization)/urdf/robotiq_arg2f_85_model_macro.xacro" />
+  <xacro:include filename="$(find realsense2_description)/urdf/_d435.urdf.xacro" />
   <xacro:property name="base_x_size" value="0.76" />
   <xacro:property name="base_y_size" value="0.46" />
@@ -44,3 +46,14 @@
     </xacro:if>
   </xacro:if>
+  <xacro:if value="$(arg realsense_enabled)">
+     <link name="realsense_base_link" />
+     <joint name="realsense_mount_fixed_joint" type="fixed">
+        <parent link="${prefix}real_ee_link"/>
+        <child link="realsense_base_link"/>
+        <origin xyz="0 0.04 0.045" rpy="0 0 ${M_PI/2}"/>
+     </joint>
+    <xacro:sensor_d435 parent="realsense_base_link" name="sensor_d435">
+      <origin xyz="0 0 0" rpy="0 0 0"/>
+    </xacro:sensor_d435>
+  </xacro:if>
 </robot>

Commit message: motion-test update

File: assembly_robot_description/urdf/rob1_gripper.urdf.xacro (robot description, xacro)
@@ -51,5 +51,5 @@
         <parent link="${prefix}real_ee_link"/>
         <child link="realsense_base_link"/>
-        <origin xyz="0 0.04 0.045" rpy="0 0 ${M_PI/2}"/>
+        <origin xyz="0 0.045 0.040" rpy="0 0 ${M_PI/2}"/>
      </joint>
     <xacro:sensor_d435 parent="realsense_base_link" name="sensor_d435">

Commit message: implement ik

File: assembly_robot_description/urdf/rob1_gripper.urdf.xacro (robot description, xacro)
@@ -34,4 +34,17 @@
     </joint>
     <link name="${prefix}real_ee_link"/>
+    <!-- for grasp point -->
+    <link name="${prefix}tcp_gripper_open"/>
+    <link name="${prefix}tcp_gripper_closed"/>
+    <joint name="${prefix}ur_tcp_fixed_joint" type="fixed">
+      <parent link="${prefix}real_ee_link"/>
+      <child link="${prefix}tcp_gripper_open"/>
+      <origin xyz="0 0 0.13" rpy="0 0 0"/>
+    </joint>
+    <joint name="${prefix}ur_gripper_closed_fixed_joint" type="fixed">
+      <parent link="${prefix}real_ee_link"/>
+      <child link="${prefix}tcp_gripper_closed"/>
+      <origin xyz="0 0 0.14" rpy="0 0 0"/>
+    </joint>
     <xacro:ur5e_robot prefix="rob1_" joint_limited="true"/>
     <!-- <xacro:ur5_robot prefix="" joint_limited="false"/> -->

File: assembly_robot_description/urdf/rob2_gripper.urdf.xacro (robot description, xacro)
@@ -33,4 +33,17 @@
     </joint>
     <link name="${prefix}real_ee_link"/>
+    <!-- for grasp point -->
+    <link name="${prefix}tcp_gripper_open"/>
+    <link name="${prefix}tcp_gripper_closed"/>
+    <joint name="${prefix}ur_tcp_fixed_joint" type="fixed">
+      <parent link="${prefix}real_ee_link"/>
+      <child link="${prefix}tcp_gripper_open"/>
+      <origin xyz="0 0 0.13" rpy="0 0 0"/>
+    </joint>
+    <joint name="${prefix}ur_gripper_closed_fixed_joint" type="fixed">
+      <parent link="${prefix}real_ee_link"/>
+      <child link="${prefix}tcp_gripper_closed"/>
+      <origin xyz="0 0 0.14" rpy="0 0 0"/>
+    </joint>
     <xacro:ur5e_robot prefix="rob2_" joint_limited="true"/>
     <!-- <xacro:ur5_robot prefix="" joint_limited="false"/> -->

Commit message: camera-motion-update

File: assembly_robot_description/urdf/rob1_gripper.urdf.xacro (robot description, xacro)
@@ -55,5 +55,5 @@
         <parent link="${prefix}tool0"/>
         <child link="${prefix}robotiq_arg2f_base_link"/>
-        <origin xyz="0 0 0" rpy="0 0 -${M_PI/2}"/>
+        <origin xyz="0 0 0.008" rpy="0 0 -${M_PI/2}"/>
       </joint>
       <xacro:robotiq_arg2f_85 prefix="rob1_"/>

File: assembly_robot_description/urdf/rob2_gripper.urdf.xacro (robot description, xacro)
@@ -53,5 +53,5 @@
         <parent link="${prefix}tool0"/>
         <child link="${prefix}robotiq_arg2f_base_link"/>
-        <origin xyz="0 0 0" rpy="0 0 -${M_PI/2}"/>
+        <origin xyz="0 0 0.008" rpy="0 0 -${M_PI/2}"/>
       </joint>
       <xacro:robotiq_arg2f_85 prefix="rob2_"/>
