Commit message: - change collision of table rod to 0.05 - add move to goal for rob2

File: assembly_robot_description/urdf/table.urdf.xacro (robot description, xacro)
@@ -15,5 +15,5 @@
          <origin xyz="0 0 0" rpy="0 0 0"/>
          <geometry>
-           <box size="0.03 0.03 1.5"/>
+           <box size="0.05 0.05 1.5"/>
          </geometry>
        </collision>
@@ -32,5 +32,5 @@
          <origin xyz="0 0 0" rpy="0 0 0"/>
          <geometry>
-           <box size="0.03 0.03 1.5"/>
+           <box size="0.05 0.05 1.5"/>
          </geometry>
        </collision>
@@ -49,5 +49,5 @@
          <origin xyz="0 0 0" rpy="0 0 0"/>
          <geometry>
-           <box size="0.03 0.03 1.5"/>
+           <box size="0.05 0.05 1.5"/>
          </geometry>
        </collision>
@@ -66,5 +66,5 @@
          <origin xyz="0 0 0" rpy="0 0 0"/>
          <geometry>
-           <box size="0.03 0.03 1.5"/>
+           <box size="0.05 0.05 1.5"/>
          </geometry>
        </collision>

Commit message: trans pc backup

File: assembly_robot_description/urdf/table.urdf.xacro (robot description, xacro)
@@ -74,5 +74,5 @@
          <origin xyz="0 0 -0.4" rpy="0 0 0" />
          <geometry>
-           <box size="1.2 2 0.8" />
+           <box size="2.3 3 0.8" />
          </geometry>
          <material name="table">
@@ -83,5 +83,5 @@
          <origin xyz="0 0 -0.4" rpy="0 0 0"/>
          <geometry>
-           <box size="1.2 1.98 0.8"/>
+           <box size="2.3 3 0.8"/>
          </geometry>
        </collision>

Commit message: update

File: assembly_robot_description/urdf/table.urdf.xacro (robot description, xacro)
@@ -15,5 +15,5 @@
          <origin xyz="0 0 0" rpy="0 0 0"/>
          <geometry>
-           <box size="0.07 0.07 1.5"/>
+           <box size="0.09 0.09 1.5"/>
          </geometry>
        </collision>
@@ -32,5 +32,5 @@
          <origin xyz="0 0 0" rpy="0 0 0"/>
          <geometry>
-           <box size="0.07 0.07 1.5"/>
+           <box size="0.09 0.09 1.5"/>
          </geometry>
        </collision>
@@ -49,5 +49,5 @@
          <origin xyz="0 0 0" rpy="0 0 0"/>
          <geometry>
-           <box size="0.07 0.07 1.5"/>
+           <box size="0.09 0.09 1.5"/>
          </geometry>
        </collision>
@@ -66,5 +66,5 @@
          <origin xyz="0 0 0" rpy="0 0 0"/>
          <geometry>
-           <box size="0.07 0.07 1.5"/>
+           <box size="0.09 0.09 1.5"/>
          </geometry>
        </collision>
@@ -86,4 +86,21 @@
          </geometry>
        </collision>
+     </link>
+    <link name="ceiling">
+      <visual>
+         <origin xyz="0 0 0.0005" rpy="0 0 0" />
+         <geometry>
+           <box size="2.3 3 0.001" />
+         </geometry>
+         <material name="ceiling">
+           <color rgba="0.192 0.192 0.192 1.0"/>
+         </material>
+       </visual>
+      <collision>
+         <origin xyz="0 0 0.0005" rpy="0 0 0"/>
+         <geometry>
+           <box size="2.3 3 0.001"/>
+         </geometry>
+      </collision>
      </link>
     <joint name="table_bar1" type="fixed">
@@ -107,3 +124,8 @@
       <origin xyz="-0.585 -0.985 0.75" rpy="0.0 0.0 0" />
     </joint>
+    <joint name="table_ceiling" type="fixed">
+      <parent link="table" />
+      <child link="ceiling" />
+      <origin xyz="0 0 1.4" rpy="0.0 0.0 0" />
+    </joint>
 </robot>

Commit message: update robot pose and table

File: assembly_robot_description/urdf/table.urdf.xacro (robot description, xacro)
@@ -70,5 +70,5 @@
        </collision>
      </link>
-    <link name="table">
+   <!--  <link name="table">
        <visual>
          <origin xyz="0 0 -0.4" rpy="0 0 0" />
@@ -84,4 +84,89 @@
          <geometry>
            <box size="2.3 3 0.8"/>
+         </geometry>
+       </collision>
+     </link> -->
+     <link name="table">
+       <visual>
+         <origin xyz="-0.885  0 -0.4" rpy="0 0 0" />
+         <geometry>
+           <box size="0.57 1.98 0.8" />
+         </geometry>
+         <material name="table">
+           <color rgba="0.192 0.192 0.192 0.7"/>
+         </material>
+       </visual>
+       <collision>
+         <origin xyz="-0.885 0 -0.4" rpy="0 0 0"/>
+         <geometry>
+           <box size="0.57 1.98 0.8"/>
+         </geometry>
+       </collision>
+     </link>
+     <link name="table_station1">
+       <visual>
+         <origin xyz="0 -0.09 -0.015" rpy="0 0 0" />
+         <geometry>
+           <box size="1.2 0.18 0.03" />
+         </geometry>
+         <material name="color1">
+           <color rgba="0.7 0.01 0.7 1.0"/>
+         </material>
+       </visual>
+       <collision>
+         <origin xyz="0 -0.09 -0.015" rpy="0 0 0"/>
+         <geometry>
+           <box size="1.2 0.18 0.8"/>
+         </geometry>
+       </collision>
+     </link>
+     <link name="table_station2">
+       <visual>
+         <origin xyz="0 0.135 -0.015" rpy="0 0 0" />
+         <geometry>
+           <box size="1.2 0.27 0.03" />
+         </geometry>
+         <material name="color2">
+           <color rgba="0.1 0.7 0.1 1.0"/>
+         </material>
+       </visual>
+       <collision>
+         <origin xyz="0 0.135 -0.015" rpy="0 0 0"/>
+         <geometry>
+           <box size="1.2 0.27 0.03"/>
+         </geometry>
+       </collision>
+     </link>
+     <link name="table_link1">
+       <visual>
+         <origin xyz="0 -0.585 -0.4" rpy="0 0 0" />
+         <geometry>
+           <box size="1.2 0.81 0.8" />
+         </geometry>
+         <material name="table">
+           <color rgba="0.192 0.192 0.192 1.0"/>
+         </material>
+       </visual>
+       <collision>
+         <origin xyz="0 -0.585 -0.4" rpy="0 0 0"/>
+         <geometry>
+           <box size="1.2 0.81 0.8"/>
+         </geometry>
+       </collision>
+     </link>
+     <link name="table_link2">
+       <visual>
+         <origin xyz="0 0.63 -0.4" rpy="0 0 0" />
+         <geometry>
+           <box size="1.2 0.72 0.8" />
+         </geometry>
+         <material name="table">
+           <color rgba="0.192 0.192 0.192 1.0"/>
+         </material>
+       </visual>
+       <collision>
+         <origin xyz="0 0.63 -0.4" rpy="0 0 0"/>
+         <geometry>
+           <box size="1.2 0.72 0.8"/>
          </geometry>
        </collision>
@@ -107,20 +192,20 @@
       <parent link="table" />
       <child link="bar1" />
-      <origin xyz="0.585 0.985 0.75" rpy="0.0 0.0 0" />
+      <origin xyz="0.990 0.985 0.75" rpy="0.0 0.0 0" />
     </joint>
     <joint name="table_bar2" type="fixed">
       <parent link="table" />
       <child link="bar2" />
-      <origin xyz="-0.585 0.985 0.75" rpy="0.0 0.0 0" />
+      <origin xyz="-1.125 0.985 0.75" rpy="0.0 0.0 0" />
     </joint>
     <joint name="table_bar3" type="fixed">
       <parent link="table" />
       <child link="bar3" />
-      <origin xyz="0.585 -0.985 0.75" rpy="0.0 0.0 0" />
+      <origin xyz="0.990 -0.985 0.75" rpy="0.0 0.0 0" />
     </joint>
     <joint name="table_bar4" type="fixed">
       <parent link="table" />
       <child link="bar4" />
-      <origin xyz="-0.585 -0.985 0.75" rpy="0.0 0.0 0" />
+      <origin xyz="-1.125 -0.985 0.75" rpy="0.0 0.0 0" />
     </joint>
     <joint name="table_ceiling" type="fixed">
@@ -129,3 +214,27 @@
       <origin xyz="0 0 1.4" rpy="0.0 0.0 0" />
     </joint>
+    <joint name="table_p_joint1" type="prismatic">
+      <parent link="table" />
+      <child link="table_station1" />
+      <origin xyz="0 0 0" rpy="0.0 0.0 0" />
+      <axis xyz="0 0 1"/>
+      <limit effort="30" velocity="1.0" lower="-1.65" upper="0.084" />
+    </joint>
+    <joint name="table_p_joint2" type="prismatic">
+      <parent link="table" />
+      <child link="table_station2" />
+      <origin xyz="0 0 0" rpy="0.0 0.0 0" />
+      <axis xyz="0 0 1"/>
+      <limit effort="30" velocity="1.0" lower="-0.028" upper="0.375" />
+    </joint>
+    <joint name="table_joint1" type="fixed">
+      <parent link="table" />
+      <child link="table_link1" />
+      <origin xyz="0 0 0" rpy="0.0 0.0 0" />
+    </joint>
+    <joint name="table_joint2" type="fixed">
+      <parent link="table" />
+      <child link="table_link2" />
+      <origin xyz="0 0 0" rpy="0.0 0.0 0" />
+    </joint>
 </robot>

Commit message: table 수치변경

File: assembly_robot_description/urdf/table.urdf.xacro (robot description, xacro)
@@ -106,14 +106,14 @@
      <link name="table_station1">
        <visual>
-         <origin xyz="0 -0.09 -0.015" rpy="0 0 0" />
+         <origin xyz="0 -0.18 -0.015" rpy="0 0 0" />
          <geometry>
            <box size="1.2 0.18 0.03" />
          </geometry>
          <material name="color1">
-           <color rgba="0.7 0.01 0.7 1.0"/>
-         </material>
-       </visual>
-       <collision>
-         <origin xyz="0 -0.09 -0.015" rpy="0 0 0"/>
+           <color rgba="0.7 0.01 0.7 0.8"/>
+         </material>
+       </visual>
+       <collision>
+         <origin xyz="0 -0.18 -0.015" rpy="0 0 0"/>
          <geometry>
            <box size="1.2 0.18 0.8"/>
@@ -123,14 +123,14 @@
      <link name="table_station2">
        <visual>
-         <origin xyz="0 0.135 -0.015" rpy="0 0 0" />
+         <origin xyz="0 0.045 -0.015" rpy="0 0 0" />
          <geometry>
            <box size="1.2 0.27 0.03" />
          </geometry>
          <material name="color2">
-           <color rgba="0.1 0.7 0.1 1.0"/>
-         </material>
-       </visual>
-       <collision>
-         <origin xyz="0 0.135 -0.015" rpy="0 0 0"/>
+           <color rgba="0.1 0.7 0.1 0.8"/>
+         </material>
+       </visual>
+       <collision>
+         <origin xyz="0 0.045 -0.015" rpy="0 0 0"/>
          <geometry>
            <box size="1.2 0.27 0.03"/>
@@ -140,5 +140,22 @@
      <link name="table_link1">
        <visual>
-         <origin xyz="0 -0.585 -0.4" rpy="0 0 0" />
+         <origin xyz="0 -0.630 -0.4" rpy="0 0 0" />
+         <geometry>
+           <box size="1.2 0.72 0.8" />
+         </geometry>
+         <material name="table">
+           <color rgba="0.192 0.192 0.192 1.0"/>
+         </material>
+       </visual>
+       <collision>
+         <origin xyz="0 -0.630 -0.4" rpy="0 0 0"/>
+         <geometry>
+           <box size="1.2 0.72 0.8"/>
+         </geometry>
+       </collision>
+     </link>
+     <link name="table_link2">
+       <visual>
+         <origin xyz="0 0.585 -0.4" rpy="0 0 0" />
          <geometry>
            <box size="1.2 0.81 0.8" />
@@ -149,24 +166,7 @@
        </visual>
        <collision>
-         <origin xyz="0 -0.585 -0.4" rpy="0 0 0"/>
+         <origin xyz="0 0.585 -0.4" rpy="0 0 0"/>
          <geometry>
            <box size="1.2 0.81 0.8"/>
-         </geometry>
-       </collision>
-     </link>
-     <link name="table_link2">
-       <visual>
-         <origin xyz="0 0.63 -0.4" rpy="0 0 0" />
-         <geometry>
-           <box size="1.2 0.72 0.8" />
-         </geometry>
-         <material name="table">
-           <color rgba="0.192 0.192 0.192 1.0"/>
-         </material>
-       </visual>
-       <collision>
-         <origin xyz="0 0.63 -0.4" rpy="0 0 0"/>
-         <geometry>
-           <box size="1.2 0.72 0.8"/>
          </geometry>
        </collision>
