Commit message: 16/10/20

File: assembly_robot_description/urdf/rob1_robot_driver.urdf.xacro (robot description, xacro)
@@ -4,5 +4,5 @@
   <xacro:arg name="ur_enabled" default="true"/>
   <xacro:arg name="gripper_enabled" default="true"/>
-  <xacro:arg name="realsense_enabled" default="true"/>
+  <xacro:arg name="realsense_enabled" default="false"/>
   <xacro:property name="M_PI" value="3.14159"/>
   <xacro:property name="base_x_size" value="0.76" />
@@ -76,3 +76,25 @@
         </xacro:sensor_d435>
     </xacro:if>
+    <joint name="${prefix}real_ee_link" type="fixed">
+      <parent link="${prefix}real_ee_link" />
+      <child link="${prefix}ELP_CAM" />
+      <origin xyz="0 0.045 0.03" rpy="0.0 0.0 0" />
+    </joint>
+    <link name="${prefix}ELP_CAM">
+       <visual>
+         <origin xyz="0 0 0.05" rpy="0 0 0" />
+         <geometry>
+           <box size="0.13 0.04 0.06" />
+         </geometry>
+         <material name="${prefix}ELP_CAM">
+           <color rgba="0.102 0.000 0.102 1.0"/>
+         </material>
+       </visual>
+       <collision>
+         <origin xyz="0 0 0.04" rpy="0 0 0"/>
+         <geometry>
+           <box size="0.13 0.05 0.06"/>
+         </geometry>
+       </collision>
+     </link>
 </robot>

File: assembly_robot_description/urdf/rob2_robot_driver.urdf.xacro (robot description, xacro)
@@ -65,4 +65,26 @@
       </xacro:if>
     </xacro:if>
+    <joint name="${prefix}real_ee_link" type="fixed">
+      <parent link="${prefix}real_ee_link" />
+      <child link="${prefix}ELP_CAM" />
+      <origin xyz="0 0.045 0.040" rpy="0.0 0.0 0" />
+    </joint>
+    <link name="${prefix}ELP_CAM">
+       <visual>
+         <origin xyz="0 0 0.05" rpy="0 0 0" />
+         <geometry>
+           <box size="0.13 0.05 0.06" />
+         </geometry>
+         <material name="${prefix}ELP_CAM">
+           <color rgba="0.102 0.000 0.102 1.0"/>
+         </material>
+       </visual>
+       <collision>
+         <origin xyz="0 0 0.05" rpy="0 0 0"/>
+         <geometry>
+           <box size="0.13 0.05 0.06"/>
+         </geometry>
+       </collision>
+     </link>
 <!--     <xacro:if value="$(arg realsense_enabled)">
        <link name="${prefix}realsense_base_link" />

File: assembly_robot_description/urdf/table.urdf.xacro (robot description, xacro)
@@ -15,5 +15,5 @@
          <origin xyz="0 0 0" rpy="0 0 0"/>
          <geometry>
-           <box size="0.05 0.05 1.5"/>
+           <box size="0.07 0.07 1.5"/>
          </geometry>
        </collision>
@@ -32,5 +32,5 @@
          <origin xyz="0 0 0" rpy="0 0 0"/>
          <geometry>
-           <box size="0.05 0.05 1.5"/>
+           <box size="0.07 0.07 1.5"/>
          </geometry>
        </collision>
@@ -49,5 +49,5 @@
          <origin xyz="0 0 0" rpy="0 0 0"/>
          <geometry>
-           <box size="0.05 0.05 1.5"/>
+           <box size="0.07 0.07 1.5"/>
          </geometry>
        </collision>
@@ -66,5 +66,5 @@
          <origin xyz="0 0 0" rpy="0 0 0"/>
          <geometry>
-           <box size="0.05 0.05 1.5"/>
+           <box size="0.07 0.07 1.5"/>
          </geometry>
        </collision>

Commit message: update

File: assembly_robot_description/urdf/rob1_robot_driver.urdf.xacro (robot description, xacro)
@@ -17,5 +17,5 @@
   <xacro:include filename="$(find robotiq_2f_85_gripper_visualization)/urdf/robotiq_arg2f_85_model_macro.xacro" />
   <!-- realsense d435 -->
-  <xacro:include filename="$(find realsense2_description)/urdf/_d435.urdf.xacro" />
+<!--   <xacro:include filename="$(find realsense2_description)/urdf/_d435.urdf.xacro" /> -->
   <!-- arm -->
   <xacro:arg name="kinematics_config" default="$(find assembly_robot_description)/config/ur5e_default.yaml"/>
@@ -65,4 +65,5 @@
       </xacro:if>
     </xacro:if>
+<!--
     <xacro:if value="$(arg realsense_enabled)">
        <link name="realsense_base_link" />
@@ -75,6 +76,6 @@
           <origin xyz="0 0 0" rpy="0 0 0"/>
         </xacro:sensor_d435>
-    </xacro:if>
-    <joint name="${prefix}real_ee_link" type="fixed">
+    </xacro:if> -->
+    <joint name="${prefix}real_ELP_link" type="fixed">
       <parent link="${prefix}real_ee_link" />
       <child link="${prefix}ELP_CAM" />
@@ -98,3 +99,69 @@
        </collision>
      </link>
+   <joint name="${prefix}safety_link" type="fixed">
+      <parent link="${prefix}real_ee_link" />
+      <child link="${prefix}safety_zone" />
+      <origin xyz="0 0 0.05" rpy="0.0 0.0 0" />
+    </joint>
+   <link name="${prefix}safety_zone">
+     <visual>
+       <origin xyz="0 0 0" rpy="0 0 0" />
+       <geometry>
+         <cylinder length="0.100" radius="0.045"/>
+       </geometry>
+       <material name="{prefix}safety_zone">
+         <color rgba="0.192 0.192 0.192 1.0"/>
+       </material>
+     </visual>
+     <collision>
+       <origin xyz="0 0 0" rpy="0 0 0"/>
+       <geometry>
+         <cylinder length="0.100" radius="0.045"/>
+       </geometry>
+     </collision>
+   </link>
+   <joint name="${prefix}safety_box1_link" type="fixed">
+      <parent link="${prefix}safety_zone" />
+      <child link="${prefix}safety_box1_zone" />
+      <origin xyz="0.07 0 0.06" rpy="0.0 0.0 0" />
+    </joint>
+   <link name="${prefix}safety_box1_zone">
+     <visual>
+       <origin xyz="0 0 0" rpy="0 0 0" />
+       <geometry>
+         <box size="0.05 0.03 0.13"/>
+       </geometry>
+       <material name="{prefix}safety_box1_zone">
+         <color rgba="0.002 0.192 0.192 1.0"/>
+       </material>
+     </visual>
+     <collision>
+       <origin xyz="0 0 0" rpy="0 0 0"/>
+       <geometry>
+         <box size="0.05 0.03 0.13"/>
+       </geometry>
+     </collision>
+   </link>
+   <joint name="${prefix}safety_box2_link" type="fixed">
+      <parent link="${prefix}safety_zone" />
+      <child link="${prefix}safety_box2_zone" />
+      <origin xyz="-0.07 0 0.06" rpy="0.0 0.0 0" />
+    </joint>
+   <link name="${prefix}safety_box2_zone">
+     <visual>
+       <origin xyz="0 0 0" rpy="0 0 0" />
+       <geometry>
+         <box size="0.05 0.03 0.13"/>
+       </geometry>
+       <material name="{prefix}safety_box2_zone">
+         <color rgba="0.002 0.192 0.192 1.0"/>
+       </material>
+     </visual>
+     <collision>
+       <origin xyz="0 0 0" rpy="0 0 0"/>
+       <geometry>
+         <box size="0.05 0.03 0.13"/>
+       </geometry>
+     </collision>
+   </link>
 </robot>

File: assembly_robot_description/urdf/rob2_robot_driver.urdf.xacro (robot description, xacro)
@@ -87,4 +87,92 @@
        </collision>
      </link>
+    <joint name="${prefix}real_sense_link" type="fixed">
+      <parent link="${prefix}real_ee_link" />
+      <child link="${prefix}sense_CAM" />
+      <origin xyz="0 -0.045 0.03" rpy="0.0 0.0 0" />
+    </joint>
+    <link name="${prefix}sense_CAM">
+       <visual>
+         <origin xyz="0 0 0.05" rpy="0 0 0" />
+         <geometry>
+           <box size="0.12 0.04 0.05" />
+         </geometry>
+         <material name="${prefix}sense_CAM">
+           <color rgba="0.102 0.000 0.102 1.0"/>
+         </material>
+       </visual>
+       <collision>
+         <origin xyz="0 0 0.04" rpy="0 0 0"/>
+         <geometry>
+           <box size="0.12 0.04 0.06"/>
+         </geometry>
+       </collision>
+     </link>
+     <joint name="${prefix}safety_link" type="fixed">
+      <parent link="${prefix}real_ee_link" />
+      <child link="${prefix}safety_zone" />
+      <origin xyz="0 0 0.05" rpy="0.0 0.0 0" />
+    </joint>
+   <link name="${prefix}safety_zone">
+     <visual>
+       <origin xyz="0 0 0" rpy="0 0 0" />
+       <geometry>
+         <cylinder length="0.100" radius="0.045"/>
+       </geometry>
+       <material name="{prefix}safety_zone">
+         <color rgba="0.192 0.192 0.192 1.0"/>
+       </material>
+     </visual>
+     <collision>
+       <origin xyz="0 0 0" rpy="0 0 0"/>
+       <geometry>
+         <cylinder length="0.100" radius="0.045"/>
+       </geometry>
+     </collision>
+   </link>
+   <joint name="${prefix}safety_box1_link" type="fixed">
+      <parent link="${prefix}safety_zone" />
+      <child link="${prefix}safety_box1_zone" />
+      <origin xyz="0.07 0 0.06" rpy="0.0 0.0 0" />
+    </joint>
+   <link name="${prefix}safety_box1_zone">
+     <visual>
+       <origin xyz="0 0 0" rpy="0 0 0" />
+       <geometry>
+         <box size="0.05 0.03 0.13"/>
+       </geometry>
+       <material name="{prefix}safety_box1_zone">
+         <color rgba="0.002 0.192 0.192 1.0"/>
+       </material>
+     </visual>
+     <collision>
+       <origin xyz="0 0 0" rpy="0 0 0"/>
+       <geometry>
+         <box size="0.05 0.03 0.13"/>
+       </geometry>
+     </collision>
+   </link>
+   <joint name="${prefix}safety_box2_link" type="fixed">
+      <parent link="${prefix}safety_zone" />
+      <child link="${prefix}safety_box2_zone" />
+      <origin xyz="-0.07 0 0.06" rpy="0.0 0.0 0" />
+    </joint>
+   <link name="${prefix}safety_box2_zone">
+     <visual>
+       <origin xyz="0 0 0" rpy="0 0 0" />
+       <geometry>
+         <box size="0.05 0.03 0.13"/>
+       </geometry>
+       <material name="{prefix}safety_box2_zone">
+         <color rgba="0.002 0.192 0.192 1.0"/>
+       </material>
+     </visual>
+     <collision>
+       <origin xyz="0 0 0" rpy="0 0 0"/>
+       <geometry>
+         <box size="0.05 0.03 0.13"/>
+       </geometry>
+     </collision>
+   </link>
 <!--     <xacro:if value="$(arg realsense_enabled)">
        <link name="${prefix}realsense_base_link" />

Commit message: 11/04update

File: assembly_robot_description/urdf/rob1_robot_driver.urdf.xacro (robot description, xacro)
@@ -124,5 +124,5 @@
       <parent link="${prefix}safety_zone" />
       <child link="${prefix}safety_box1_zone" />
-      <origin xyz="0.07 0 0.06" rpy="0.0 0.0 0" />
+      <origin xyz="0.05 0 0.06" rpy="0.0 0.0 0" />
     </joint>
    <link name="${prefix}safety_box1_zone">
@@ -130,5 +130,5 @@
        <origin xyz="0 0 0" rpy="0 0 0" />
        <geometry>
-         <box size="0.05 0.03 0.13"/>
+         <box size="0.02 0.05 0.13"/>
        </geometry>
        <material name="{prefix}safety_box1_zone">
@@ -139,5 +139,5 @@
        <origin xyz="0 0 0" rpy="0 0 0"/>
        <geometry>
-         <box size="0.05 0.03 0.13"/>
+         <box size="0.02 0.05 0.13"/>
        </geometry>
      </collision>
@@ -146,5 +146,5 @@
       <parent link="${prefix}safety_zone" />
       <child link="${prefix}safety_box2_zone" />
-      <origin xyz="-0.07 0 0.06" rpy="0.0 0.0 0" />
+      <origin xyz="-0.05 0 0.06" rpy="0.0 0.0 0" />
     </joint>
    <link name="${prefix}safety_box2_zone">
@@ -152,5 +152,5 @@
        <origin xyz="0 0 0" rpy="0 0 0" />
        <geometry>
-         <box size="0.05 0.03 0.13"/>
+         <box size="0.02 0.05 0.13"/>
        </geometry>
        <material name="{prefix}safety_box2_zone">
@@ -161,5 +161,5 @@
        <origin xyz="0 0 0" rpy="0 0 0"/>
        <geometry>
-         <box size="0.05 0.03 0.13"/>
+         <box size="0.02 0.05 0.13"/>
        </geometry>
      </collision>

File: assembly_robot_description/urdf/rob2_robot_driver.urdf.xacro (robot description, xacro)
@@ -134,5 +134,5 @@
       <parent link="${prefix}safety_zone" />
       <child link="${prefix}safety_box1_zone" />
-      <origin xyz="0.07 0 0.06" rpy="0.0 0.0 0" />
+      <origin xyz="0.05 0 0.06" rpy="0.0 0.0 0" />
     </joint>
    <link name="${prefix}safety_box1_zone">
@@ -140,5 +140,5 @@
        <origin xyz="0 0 0" rpy="0 0 0" />
        <geometry>
-         <box size="0.05 0.03 0.13"/>
+         <box size="0.02 0.05 0.13"/>
        </geometry>
        <material name="{prefix}safety_box1_zone">
@@ -149,5 +149,5 @@
        <origin xyz="0 0 0" rpy="0 0 0"/>
        <geometry>
-         <box size="0.05 0.03 0.13"/>
+         <box size="0.02 0.05 0.13"/>
        </geometry>
      </collision>
@@ -156,5 +156,5 @@
       <parent link="${prefix}safety_zone" />
       <child link="${prefix}safety_box2_zone" />
-      <origin xyz="-0.07 0 0.06" rpy="0.0 0.0 0" />
+      <origin xyz="-0.05 0 0.06" rpy="0.0 0.0 0" />
     </joint>
    <link name="${prefix}safety_box2_zone">
@@ -162,5 +162,5 @@
        <origin xyz="0 0 0" rpy="0 0 0" />
        <geometry>
-         <box size="0.05 0.03 0.13"/>
+         <box size="0.02 0.05 0.13"/>
        </geometry>
        <material name="{prefix}safety_box2_zone">
@@ -171,5 +171,5 @@
        <origin xyz="0 0 0" rpy="0 0 0"/>
        <geometry>
-         <box size="0.05 0.03 0.13"/>
+         <box size="0.02 0.05 0.13"/>
        </geometry>
      </collision>

Commit message: backup update

File: assembly_robot_description/urdf/rob1_robot_driver.urdf.xacro (robot description, xacro)
@@ -122,44 +122,46 @@
    </link>
    <joint name="${prefix}safety_box1_link" type="fixed">
-      <parent link="${prefix}safety_zone" />
+      <!-- <parent link="${prefix}safety_zone" /> -->
+      <parent link="${prefix}right_inner_finger_pad" />
       <child link="${prefix}safety_box1_zone" />
-      <origin xyz="0.05 0 0.06" rpy="0.0 0.0 0" />
+      <origin xyz="0.0 0 0.0" rpy="0.0 0.0 0" />
     </joint>
    <link name="${prefix}safety_box1_zone">
      <visual>
-       <origin xyz="0 0 0" rpy="0 0 0" />
+       <origin xyz="0 0.02 0" rpy="0 0 0" />
        <geometry>
-         <box size="0.02 0.05 0.13"/>
+         <box size="0.05 0.02 0.08"/>
        </geometry>
        <material name="{prefix}safety_box1_zone">
-         <color rgba="0.002 0.192 0.192 1.0"/>
+         <color rgba="0.002 0.192 0.192 0.5"/>
        </material>
      </visual>
      <collision>
-       <origin xyz="0 0 0" rpy="0 0 0"/>
+       <origin xyz="0 0.02 0" rpy="0 0 0"/>
        <geometry>
-         <box size="0.02 0.05 0.13"/>
+         <box size="0.05 0.04 0.01"/>
        </geometry>
      </collision>
    </link>
    <joint name="${prefix}safety_box2_link" type="fixed">
-      <parent link="${prefix}safety_zone" />
+      <!-- <parent link="${prefix}safety_zone" /> -->
+      <parent link="${prefix}left_inner_finger_pad" />
       <child link="${prefix}safety_box2_zone" />
-      <origin xyz="-0.05 0 0.06" rpy="0.0 0.0 0" />
+      <origin xyz="0.00 0 0.0" rpy="0.0 0.0 0" />
     </joint>
    <link name="${prefix}safety_box2_zone">
      <visual>
-       <origin xyz="0 0 0" rpy="0 0 0" />
+       <origin xyz="0 0.02 0" rpy="0 0 0" />
        <geometry>
-         <box size="0.02 0.05 0.13"/>
+         <box size="0.05 0.02 0.08"/>
        </geometry>
        <material name="{prefix}safety_box2_zone">
-         <color rgba="0.002 0.192 0.192 1.0"/>
+         <color rgba="0.002 0.192 0.192 0.5"/>
        </material>
      </visual>
      <collision>
-       <origin xyz="0 0 0" rpy="0 0 0"/>
+       <origin xyz="0 0.02 0" rpy="0 0 0"/>
        <geometry>
-         <box size="0.02 0.05 0.13"/>
+         <box size="0.05 0.04 0.01"/>
        </geometry>
      </collision>

File: assembly_robot_description/urdf/rob2_robot_driver.urdf.xacro (robot description, xacro)
@@ -132,7 +132,8 @@
    </link>
    <joint name="${prefix}safety_box1_link" type="fixed">
-      <parent link="${prefix}safety_zone" />
+      <!-- <parent link="${prefix}safety_zone" /> -->
+      <parent link="${prefix}right_inner_finger_pad" />
       <child link="${prefix}safety_box1_zone" />
-      <origin xyz="0.05 0 0.06" rpy="0.0 0.0 0" />
+      <origin xyz="0.0 0 0" rpy="0.0 0.0 0" />
     </joint>
    <link name="${prefix}safety_box1_zone">
@@ -140,5 +141,5 @@
        <origin xyz="0 0 0" rpy="0 0 0" />
        <geometry>
-         <box size="0.02 0.05 0.13"/>
+         <box size="0.05 0.02 0.13"/>
        </geometry>
        <material name="{prefix}safety_box1_zone">
@@ -149,12 +150,13 @@
        <origin xyz="0 0 0" rpy="0 0 0"/>
        <geometry>
-         <box size="0.02 0.05 0.13"/>
+         <box size="0.05 0.02 0.01"/>
        </geometry>
      </collision>
    </link>
    <joint name="${prefix}safety_box2_link" type="fixed">
-      <parent link="${prefix}safety_zone" />
+      <!-- <parent link="${prefix}safety_zone" /> -->
+      <parent link="${prefix}left_inner_finger_pad" />
       <child link="${prefix}safety_box2_zone" />
-      <origin xyz="-0.05 0 0.06" rpy="0.0 0.0 0" />
+      <origin xyz="0 0 0" rpy="0.0 0.0 0" />
     </joint>
    <link name="${prefix}safety_box2_zone">
@@ -162,5 +164,5 @@
        <origin xyz="0 0 0" rpy="0 0 0" />
        <geometry>
-         <box size="0.02 0.05 0.13"/>
+         <box size="0.05 0.02 0.13"/>
        </geometry>
        <material name="{prefix}safety_box2_zone">
@@ -171,5 +173,5 @@
        <origin xyz="0 0 0" rpy="0 0 0"/>
        <geometry>
-         <box size="0.02 0.05 0.13"/>
+         <box size="0.05 0.02 0.01"/>
        </geometry>
      </collision>

File: assembly_robot_description/urdf/table.urdf.xacro (robot description, xacro)
@@ -104,5 +104,5 @@
        </collision>
      </link>
-     <link name="table_station1">
+     <link name="table_station2">
        <visual>
          <origin xyz="0 -0.18 -0.015" rpy="0 0 0" />
@@ -117,9 +117,9 @@
          <origin xyz="0 -0.18 -0.015" rpy="0 0 0"/>
          <geometry>
-           <box size="1.2 0.18 0.8"/>
-         </geometry>
-       </collision>
-     </link>
-     <link name="table_station2">
+           <box size="1.2 0.18 0.03"/>
+         </geometry>
+       </collision>
+     </link>
+     <link name="table_station1">
        <visual>
          <origin xyz="0 0.045 -0.015" rpy="0 0 0" />
@@ -214,14 +214,14 @@
       <origin xyz="0 0 1.4" rpy="0.0 0.0 0" />
     </joint>
-    <joint name="table_p_joint1" type="prismatic">
-      <parent link="table" />
-      <child link="table_station1" />
+    <joint name="table_p_joint2" type="prismatic">
+      <parent link="table" />
+      <child link="table_station2" />
       <origin xyz="0 0 0" rpy="0.0 0.0 0" />
       <axis xyz="0 0 1"/>
       <limit effort="30" velocity="1.0" lower="-1.65" upper="0.084" />
     </joint>
-    <joint name="table_p_joint2" type="prismatic">
-      <parent link="table" />
-      <child link="table_station2" />
+    <joint name="table_p_joint1" type="prismatic">
+      <parent link="table" />
+      <child link="table_station1" />
       <origin xyz="0 0 0" rpy="0.0 0.0 0" />
       <axis xyz="0 0 1"/>
