Commit message: multi-robot-moveit-setup update

File: assembly_robot_description/urdf/rob1_rob2_multiarm.urdf.xacro (robot description, xacro)
@@ -4,16 +4,16 @@
     <xacro:include filename="$(find assembly_robot_description)/urdf/rob1_gripper.urdf.xacro" />
     <xacro:include filename="$(find assembly_robot_description)/urdf/rob2_gripper.urdf.xacro" />
-    <link name="world"/>
+    <xacro:include filename="$(find assembly_robot_description)/urdf/table.urdf.xacro" />
     <joint name = "rob1_robot_body" type = "fixed">
-        <parent link = "world"/>
+        <parent link = "table"/>
         <child link = "rob1_world"/>
         <axis xyz = "0 0 0"/>
-        <origin xyz = "0 0.11 0" rpy = "0 0 0"/>
+        <origin xyz = "0 0.76 0.01" rpy = "0 0 0"/>
     </joint>
     <joint name = "rob2_robot_body" type = "fixed">
-        <parent link = "world"/>
+        <parent link = "table"/>
         <child link = "rob2_world"/>
         <axis xyz = "0 0 0"/>
-        <origin xyz = "0 -0.11 0" rpy = "0 0 0"/>
+        <origin xyz = "0 -0.76 0.01" rpy = "0 0 ${M_PI}"/>
     </joint>
 </robot>

Commit message: world frame update

File: assembly_robot_description/urdf/rob1_rob2_multiarm.urdf.xacro (robot description, xacro)
@@ -5,4 +5,10 @@
     <xacro:include filename="$(find assembly_robot_description)/urdf/rob2_gripper.urdf.xacro" />
     <xacro:include filename="$(find assembly_robot_description)/urdf/table.urdf.xacro" />
+    <link name="world"/>
+    <joint name="world_table" type="fixed">
+        <parent link="world" />
+        <child link="table" />
+        <origin xyz="0 0.0 0.8" rpy="0.0 0.0 0" />
+    </joint>
     <joint name = "rob1_robot_body" type = "fixed">
         <parent link = "table"/>

Commit message: disinable collision check update

File: assembly_robot_description/urdf/rob1_rob2_multiarm.urdf.xacro (robot description, xacro)
@@ -15,5 +15,5 @@
         <child link = "rob1_world"/>
         <axis xyz = "0 0 0"/>
-        <origin xyz = "0 0.76 0.01" rpy = "0 0 0"/>
+        <origin xyz = "0 0.745 0.01" rpy = "0 0 0"/>
     </joint>
     <joint name = "rob2_robot_body" type = "fixed">
@@ -21,5 +21,5 @@
         <child link = "rob2_world"/>
         <axis xyz = "0 0 0"/>
-        <origin xyz = "0 -0.76 0.01" rpy = "0 0 ${M_PI}"/>
+        <origin xyz = "0 -0.685 0.01" rpy = "0 0 ${M_PI}"/>
     </joint>
 </robot>

Commit message: service update

File: assembly_robot_description/urdf/rob1_rob2_multiarm.urdf.xacro (robot description, xacro)
@@ -23,3 +23,9 @@
         <origin xyz = "0 -0.685 0.01" rpy = "0 0 ${M_PI}"/>
     </joint>
+    <link name="basler_camera"/>
+    <joint name="basler_joint" type="fixed">
+        <parent link="rob1_real_ee_link" />
+        <child link="basler_camera" />
+        <origin xyz="0 0.0 0.1" rpy="0.0 0.0 -1.5707" />
+    </joint>
 </robot>

Commit message: update

File: assembly_robot_description/urdf/rob1_rob2_multiarm.urdf.xacro (robot description, xacro)
@@ -23,9 +23,9 @@
         <origin xyz = "0 -0.685 0.01" rpy = "0 0 ${M_PI}"/>
     </joint>
-    <link name="basler_camera"/>
+    <link name="camera_center"/>
     <joint name="basler_joint" type="fixed">
         <parent link="rob1_real_ee_link" />
-        <child link="basler_camera" />
-        <origin xyz="0 0.0 0.1" rpy="0.0 0.0 -1.5707" />
+        <child link="camera_center" />
+        <origin xyz="0 0.05785 0.0721" rpy="1.5707 0 0" />
     </joint>
 </robot>

Commit message: 0911-update

File: assembly_robot_description/urdf/rob1_rob2_multiarm.urdf.xacro (robot description, xacro)
@@ -23,8 +23,14 @@
         <origin xyz = "0 -0.685 0.01" rpy = "0 0 ${M_PI}"/>
     </joint>
-    <link name="camera_center"/>
+    <link name="camera_center_1"/>
     <joint name="basler_joint" type="fixed">
         <parent link="rob1_real_ee_link" />
-        <child link="camera_center" />
+        <child link="camera_center_1" />
+        <origin xyz="0 0.05785 0.0721" rpy="1.5707 0 0" />
+    </joint>
+    <link name="camera_center_2"/>
+    <joint name="basler_joint_2" type="fixed">
+        <parent link="rob2_real_ee_link" />
+        <child link="camera_center_2" />
         <origin xyz="0 0.05785 0.0721" rpy="1.5707 0 0" />
     </joint>

Commit message: chan control

File: assembly_robot_description/urdf/rob1_rob2_multiarm.urdf.xacro (robot description, xacro)
@@ -15,5 +15,5 @@
         <child link = "rob1_world"/>
         <axis xyz = "0 0 0"/>
-        <origin xyz = "0 0.745 0.01" rpy = "0 0 0"/>
+        <origin xyz = "-0.004 0.750 0.01" rpy = "0 0 0"/>
     </joint>
     <joint name = "rob2_robot_body" type = "fixed">
@@ -21,5 +21,5 @@
         <child link = "rob2_world"/>
         <axis xyz = "0 0 0"/>
-        <origin xyz = "0 -0.685 0.01" rpy = "0 0 ${M_PI}"/>
+        <origin xyz = "0.00 -0.690 0.01" rpy = "0 0 ${M_PI}"/>
     </joint>
     <link name="camera_center_1"/>

File: assembly_robot_description/urdf/table.urdf.xacro (robot description, xacro)
@@ -83,5 +83,5 @@
          <origin xyz="0 0 -0.4" rpy="0 0 0"/>
          <geometry>
-           <box size="1.2 2 0.8"/>
+           <box size="1.2 1.98 0.8"/>
          </geometry>
        </collision>

Commit message: hole-update

File: assembly_robot_description/urdf/rob1_rob2_multiarm.urdf.xacro (robot description, xacro)
@@ -35,3 +35,9 @@
         <origin xyz="0 0.05785 0.0721" rpy="1.5707 0 0" />
     </joint>
+    <link name="screw_tool_link"/>
+    <joint name="screw_tool_joint" type="fixed">
+        <parent link="rob1_real_ee_link" />
+        <child link="screw_tool_link" />
+        <origin xyz="0 0.1115 0.144" rpy="-1.5707 -1.5707 0" />
+    </joint>
 </robot>

Commit message: update

File: assembly_robot_description/urdf/rob1_rob2_multiarm.urdf.xacro (robot description, xacro)
@@ -9,5 +9,5 @@
         <parent link="world" />
         <child link="table" />
-        <origin xyz="0 0.0 0.8" rpy="0.0 0.0 0" />
+        <origin xyz="00 0.0 0.8" rpy="0.0 0.0 0" />
     </joint>
     <joint name = "rob1_robot_body" type = "fixed">
@@ -15,5 +15,5 @@
         <child link = "rob1_world"/>
         <axis xyz = "0 0 0"/>
-        <origin xyz = "-0.004 0.750 0.01" rpy = "0 0 0"/>
+        <origin xyz = "0.096 0.750 0.01" rpy = "0 0 0"/>
     </joint>
     <joint name = "rob2_robot_body" type = "fixed">
@@ -21,5 +21,5 @@
         <child link = "rob2_world"/>
         <axis xyz = "0 0 0"/>
-        <origin xyz = "0.00 -0.690 0.01" rpy = "0 0 ${M_PI}"/>
+        <origin xyz = "0.10 -0.690 0.01" rpy = "0 0 ${M_PI}"/>
     </joint>
     <link name="camera_center_1"/>

Commit message: robot pose update

File: assembly_robot_description/urdf/rob1_rob2_multiarm.urdf.xacro (robot description, xacro)
@@ -21,5 +21,5 @@
         <child link = "rob2_world"/>
         <axis xyz = "0 0 0"/>
-        <origin xyz = "0.10 -0.690 0.01" rpy = "0 0 ${M_PI}"/>
+        <origin xyz = "0.10 -0.630 0.01" rpy = "0 0 ${M_PI}"/>
     </joint>
     <link name="camera_center_1"/>

Commit message: update 로봇 안움직임

File: assembly_robot_description/urdf/rob1_rob2_multiarm.urdf.xacro (robot description, xacro)
@@ -5,4 +5,5 @@
     <xacro:include filename="$(find assembly_robot_description)/urdf/rob2_robot_driver.urdf.xacro" />
     <xacro:include filename="$(find assembly_robot_description)/urdf/table.urdf.xacro" />
+    <!-- <xacro:include filename="$(find assembly_robot_description)/urdf/station.xacro" /> -->
     <link name="world"/>
     <joint name="world_table" type="fixed">
@@ -41,3 +42,8 @@
         <origin xyz="0 0.1115 0.144" rpy="-1.5707 -1.5707 0" />
     </joint>
+    <!-- <joint name="station_joint" type="fixed">
+        <parent link="table"/>
+        <child link="station_base_link"/>
+        <origin xyz="0.825 0 -0.455" rpy="0 0 3.14"/>
+    </joint> -->
 </robot>

Commit message: update backup

File: assembly_robot_description/urdf/rob1_rob2_multiarm.urdf.xacro (robot description, xacro)
@@ -5,5 +5,5 @@
     <xacro:include filename="$(find assembly_robot_description)/urdf/rob2_robot_driver.urdf.xacro" />
     <xacro:include filename="$(find assembly_robot_description)/urdf/table.urdf.xacro" />
-    <!-- <xacro:include filename="$(find assembly_robot_description)/urdf/station.xacro" /> -->
+    <xacro:include filename="$(find assembly_robot_description)/urdf/station.xacro" />
     <link name="world"/>
     <joint name="world_table" type="fixed">
@@ -42,8 +42,8 @@
         <origin xyz="0 0.1115 0.144" rpy="-1.5707 -1.5707 0" />
     </joint>
-    <!-- <joint name="station_joint" type="fixed">
+    <joint name="station_joint" type="fixed">
         <parent link="table"/>
         <child link="station_base_link"/>
         <origin xyz="0.825 0 -0.455" rpy="0 0 3.14"/>
-    </joint> -->
+    </joint>
 </robot>

Commit message: update

File: assembly_robot_description/urdf/rob1_rob2_multiarm.urdf.xacro (robot description, xacro)
@@ -26,7 +26,8 @@
     <link name="camera_center_1"/>
     <joint name="basler_joint" type="fixed">
-        <parent link="rob1_real_ee_link" />
+        <!-- <parent link="rob1_real_ee_link" / -->>
+        <parent link="rob1_robotiq_arg2f_base_link" />
         <child link="camera_center_1" />
-        <origin xyz="0 0.05785 0.0721" rpy="1.5707 0 0" />
+        <origin xyz="-0.05785 0 0.06386" rpy="-1.5707 3.1415 -1.5707" />
     </joint>
     <link name="camera_center_2"/>

Commit message: table control update

File: assembly_robot_description/urdf/rob1_rob2_multiarm.urdf.xacro (robot description, xacro)
@@ -26,8 +26,8 @@
     <link name="camera_center_1"/>
     <joint name="basler_joint" type="fixed">
-        <!-- <parent link="rob1_real_ee_link" / -->>
-        <parent link="rob1_robotiq_arg2f_base_link" />
+        <parent link="rob1_real_ee_link" />
+        <!-- <parent link="rob1_robotiq_arg2f_base_link" /> -->
         <child link="camera_center_1" />
-        <origin xyz="-0.05785 0 0.06386" rpy="-1.5707 3.1415 -1.5707" />
+        <origin xyz="0 0.05785 0.0721" rpy="1.5707 0 0" />
     </joint>
     <link name="camera_center_2"/>
@@ -37,8 +37,14 @@
         <origin xyz="0 0.05785 0.0721" rpy="1.5707 0 0" />
     </joint>
-    <link name="screw_tool_link"/>
-    <joint name="screw_tool_joint" type="fixed">
+    <link name="rob1_screw_tool_link"/>
+    <joint name="rob1_screw_tool_joint" type="fixed">
         <parent link="rob1_real_ee_link" />
-        <child link="screw_tool_link" />
+        <child link="rob1_screw_tool_link" />
+        <origin xyz="0 0.1115 0.144" rpy="-1.5707 -1.5707 0" />
+    </joint>
+    <link name="rob2_screw_tool_link"/>
+    <joint name="rob2_screw_tool_joint" type="fixed">
+        <parent link="rob2_real_ee_link" />
+        <child link="rob2_screw_tool_link" />
         <origin xyz="0 0.1115 0.144" rpy="-1.5707 -1.5707 0" />
     </joint>

Commit message: update code

File: assembly_robot_description/urdf/rob1_rob2_multiarm.urdf.xacro (robot description, xacro)
@@ -41,5 +41,5 @@
         <parent link="rob1_real_ee_link" />
         <child link="rob1_screw_tool_link" />
-        <origin xyz="0 0.1115 0.144" rpy="-1.5707 -1.5707 0" />
+        <origin xyz="0 -0.1115 0.144" rpy="-1.5707 -1.5707 3.1415" />
     </joint>
     <link name="rob2_screw_tool_link"/>
@@ -47,5 +47,5 @@
         <parent link="rob2_real_ee_link" />
         <child link="rob2_screw_tool_link" />
-        <origin xyz="0 0.1115 0.144" rpy="-1.5707 -1.5707 0" />
+        <origin xyz="0 -0.1115 0.144" rpy="-1.5707 -1.5707 3.1415" />
     </joint>
     <joint name="station_joint" type="fixed">

Commit message: 로봇 위치 변경

File: assembly_robot_description/urdf/rob1_rob2_multiarm.urdf.xacro (robot description, xacro)
@@ -16,5 +16,5 @@
         <child link = "rob1_world"/>
         <axis xyz = "0 0 0"/>
-        <origin xyz = "0.096 0.750 0.01" rpy = "0 0 0"/>
+        <origin xyz = "0.096 0.810 0.01" rpy = "0 0 0"/>
     </joint>
     <joint name = "rob2_robot_body" type = "fixed">
@@ -22,5 +22,5 @@
         <child link = "rob2_world"/>
         <axis xyz = "0 0 0"/>
-        <origin xyz = "0.10 -0.630 0.01" rpy = "0 0 ${M_PI}"/>
+        <origin xyz = "0.10 -0.690 0.01" rpy = "0 0 ${M_PI}"/>
     </joint>
     <link name="camera_center_1"/>
